Commit message: Got it reading off the follower bot correctly, very close, just need some tuning on the params

File: src/lerobot_description/urdf/so101.urdf.xacro (robot description, xacro)
@@ -3,4 +3,6 @@
     <xacro:arg name="use_sim" default="true"/>
     <xacro:arg name="usb_port" default="/dev/so101_follower"/>
+    <!-- Hardware: state-only ros2_control joints → Feetech driver disables torque (see feetech_ros2_driver on_init). -->
+    <xacro:arg name="hardware_passive" default="false"/>
     <xacro:include filename="$(find lerobot_description)/urdf/so101_base.xacro"/>
     <xacro:if value="${'$(arg use_sim)' in ('true', 'True', '1', 'yes')}">

File: src/lerobot_description/urdf/so101_base.xacro (robot description, xacro)
@@ -20,15 +20,19 @@
 		<color rgba="0.1 0.1 0.1 1.0" />
 	</material>
-	<!-- Link base -->
+	<!--
+	  Base link matches SO-ARM100 Simulation/SO101/so101_new_calib.urdf (Onshape export).
+	  A mismatched base link frame vs shoulder_pan made the arm look twisted in RViz while
+	  downstream link meshes already matched that reference.
+	-->
 	<link name="base">
 		<inertial>
-			<origin xyz="0.020739 0.00204287 0.065966" rpy="0 0 0" />
+			<origin xyz="0.0137179 -5.19711e-05 0.0334843" rpy="0 0 0" />
 			<mass value="0.147" />
-			<inertia ixx="0.000136117" ixy="4.59787e-07" ixz="9.75275e-08" iyy="0.000114686"
-				iyz="-4.97151e-06" izz="0.000130364" />
+			<inertia ixx="0.000114686" ixy="-4.59787e-07" ixz="4.97151e-06" iyy="0.000136117"
+				iyz="9.75275e-08" izz="0.000130364" />
 		</inertial>
 		<!-- Part base_motor_holder_so101_v1 -->
 		<visual>
-			<origin xyz="0.0206915 0.0221255 0.0300817" rpy="1.5708 -1.23909e-16 2.33147e-15" />
+			<origin xyz="-0.00636471 -9.94414e-05 -0.0024" rpy="1.5708 -1.67685e-15 1.5708" />
 			<geometry>
 				<mesh
@@ -38,5 +42,5 @@
 		</visual>
 		<collision>
-			<origin xyz="0.0206915 0.0221255 0.0300817" rpy="1.5708 -1.23909e-16 2.33147e-15" />
+			<origin xyz="-0.00636471 -9.94414e-05 -0.0024" rpy="1.5708 -1.67685e-15 1.5708" />
 			<geometry>
 				<mesh
@@ -46,5 +50,5 @@
 		<!-- Part base_so101_v2 -->
 		<visual>
-			<origin xyz="0.0207909 0.0221255 0.0300817" rpy="1.5708 -0 0" />
+			<origin xyz="-0.00636471 -8.97657e-09 -0.0024" rpy="1.5708 -2.78073e-29 1.5708" />
 			<geometry>
 				<mesh filename="package://lerobot_description/meshes/so101/base_so101_v2.stl" />
@@ -53,5 +57,5 @@
 		</visual>
 		<collision>
-			<origin xyz="0.0207909 0.0221255 0.0300817" rpy="1.5708 -0 0" />
+			<origin xyz="-0.00636471 -8.97657e-09 -0.0024" rpy="1.5708 -2.78073e-29 1.5708" />
 			<geometry>
 				<mesh filename="package://lerobot_description/meshes/so101/base_so101_v2.stl" />
@@ -60,12 +64,12 @@
 		<!-- Part sts3215_03a_v1 -->
 		<visual>
-			<origin xyz="0.0207909 -0.0105745 0.0761817" rpy="-2.20282e-15 2.77556e-17 -1.5708" />
-			<geometry>
-				<mesh filename="package://lerobot_description/meshes/so101/sts3215_03a_v1.stl" />
-			</geometry>
-			<material name="sts3215" />
-		</visual>
-		<collision>
-			<origin xyz="0.0207909 -0.0105745 0.0761817" rpy="-2.20282e-15 2.77556e-17 -1.5708" />
+			<origin xyz="0.0263353 -8.97657e-09 0.0437" rpy="-8.21148e-16 7.84513e-18 1.249e-15" />
+			<geometry>
+				<mesh filename="package://lerobot_description/meshes/so101/sts3215_03a_v1.stl" />
+			</geometry>
+			<material name="sts3215" />
+		</visual>
+		<collision>
+			<origin xyz="0.0263353 -8.97657e-09 0.0437" rpy="-8.21148e-16 7.84513e-18 1.249e-15" />
 			<geometry>
 				<mesh filename="package://lerobot_description/meshes/so101/sts3215_03a_v1.stl" />
@@ -74,5 +78,5 @@
 		<!-- Part waveshare_mounting_plate_so101_v2 -->
 		<visual>
-			<origin xyz="0.0205915 0.0467435 0.0798817" rpy="1.5708 -1.21716e-14 2.33147e-15" />
+			<origin xyz="-0.0309827 -0.000199441 0.0474" rpy="1.5708 -1.35493e-14 1.5708" />
 			<geometry>
 				<mesh
@@ -82,5 +86,5 @@
 		</visual>
 		<collision>
-			<origin xyz="0.0205915 0.0467435 0.0798817" rpy="1.5708 -1.21716e-14 2.33147e-15" />
+			<origin xyz="-0.0309827 -0.000199441 0.0474" rpy="1.5708 -1.35493e-14 1.5708" />
 			<geometry>
 				<mesh
@@ -349,17 +353,7 @@
 		<limit effort="10" velocity="10" lower="-0.22" upper="1.74533" />
 	</joint>
-	<transmission name="gripper_joint_trans">
-		<type>transmission_interface/SimpleTransmission</type>
-		<joint name="gripper_joint">
-			<hardwareInterface>hardware_interface/PositionJointInterface</hardwareInterface>
-		</joint>
-		<actuator name="motor6">
-			<hardwareInterface>hardware_interface/PositionJointInterface</hardwareInterface>
-			<mechanicalReduction>1</mechanicalReduction>
-		</actuator>
-	</transmission>
 	<!-- Joint from wrist to gripper link -->
 	<joint name="wrist_roll" type="revolute">
-		<origin xyz="0 -0.0611 0.0181" rpy="1.5708 -9.38083e-08 3.14159" />
+		<origin xyz="5.55112e-17 -0.0611 0.0181" rpy="1.5708 0.0486795 3.14159" />
 		<parent link="wrist" />
 		<child link="gripper" />
@@ -367,14 +361,4 @@
 		<limit effort="10" velocity="10" lower="-2.79253" upper="2.79253" />
 	</joint>
-	<transmission name="wrist_roll_trans">
-		<type>transmission_interface/SimpleTransmission</type>
-		<joint name="wrist_roll">
-			<hardwareInterface>hardware_interface/PositionJointInterface</hardwareInterface>
-		</joint>
-		<actuator name="motor5">
-			<hardwareInterface>hardware_interface/PositionJointInterface</hardwareInterface>
-			<mechanicalReduction>1</mechanicalReduction>
-		</actuator>
-	</transmission>
 	<!-- Joint from lower_arm to wrist -->
 	<joint name="wrist_flex" type="revolute">
@@ -385,14 +369,4 @@
 		<limit effort="10" velocity="10" lower="-1.65806" upper="1.65806" />
 	</joint>
-	<transmission name="wrist_flex_trans">
-		<type>transmission_interface/SimpleTransmission</type>
-		<joint name="wrist_flex">
-			<hardwareInterface>hardware_interface/PositionJointInterface</hardwareInterface>
-		</joint>
-		<actuator name="motor4">
-			<hardwareInterface>hardware_interface/PositionJointInterface</hardwareInterface>
-			<mechanicalReduction>1</mechanicalReduction>
-		</actuator>
-	</transmission>
 	<!-- Joint from upper_arm to lower_arm -->
 	<joint name="elbow_flex" type="revolute">
@@ -404,14 +378,4 @@
 		<limit effort="10" velocity="10" lower="-1.74533" upper="1.85" />
 	</joint>
-	<transmission name="elbow_flex_trans">
-		<type>transmission_interface/SimpleTransmission</type>
-		<joint name="elbow_flex">
-			<hardwareInterface>hardware_interface/PositionJointInterface</hardwareInterface>
-		</joint>
-		<actuator name="motor3">
-			<hardwareInterface>hardware_interface/PositionJointInterface</hardwareInterface>
-			<mechanicalReduction>1</mechanicalReduction>
-		</actuator>
-	</transmission>
 	<!-- Joint from shoulder to upper_arm -->
 	<joint name="shoulder_lift" type="revolute">
@@ -422,17 +386,7 @@
 		<limit effort="10" velocity="10" lower="-2.05" upper="1.74533" />
 	</joint>
-	<transmission name="shoulder_lift_trans">
-		<type>transmission_interface/SimpleTransmission</type>
-		<joint name="shoulder_lift">
-			<hardwareInterface>hardware_interface/PositionJointInterface</hardwareInterface>
-		</joint>
-		<actuator name="motor2">
-			<hardwareInterface>hardware_interface/PositionJointInterface</hardwareInterface>
-			<mechanicalReduction>1</mechanicalReduction>
-		</actuator>
-	</transmission>
 	<!-- Joint from base to shoulder -->
 	<joint name="shoulder_pan" type="revolute">
-		<origin xyz="0.0207909 -0.0230745 0.0948817" rpy="-3.14159 6.03684e-16 1.5708" />
+		<origin xyz="0.0388353 -8.97657e-09 0.0624" rpy="3.14159 4.18253e-17 -3.14159" />
 		<parent link="base" />
 		<child link="shoulder" />
@@ -440,13 +394,3 @@
 		<limit effort="10" velocity="10" lower="-1.91986" upper="1.91986" />
 	</joint>
-	<transmission name="shoulder_pan_trans">
-		<type>transmission_interface/SimpleTransmission</type>
-		<joint name="shoulder_pan">
-			<hardwareInterface>hardware_interface/PositionJointInterface</hardwareInterface>
-		</joint>
-		<actuator name="motor1">
-			<hardwareInterface>hardware_interface/PositionJointInterface</hardwareInterface>
-			<mechanicalReduction>1</mechanicalReduction>
-		</actuator>
-	</transmission>
 </robot>

File: src/lerobot_description/urdf/so101_ros2_control.xacro (robot description, xacro)
@@ -4,6 +4,49 @@
     <xacro:arg name="use_sim" default="true"/>
     <xacro:arg name="usb_port" default="/dev/so101_follower"/>
-    <!-- Homing offsets from config/robots/so_follower/gi_jane.json (Feetech raw encoder). -->
+    <xacro:arg name="hardware_passive" default="false"/>
+    <!--
+      Hardware calibration: config/so101_follower_calibration.yaml (xacro.load_yaml).
+      Export LeRobot gi_jane.json via python3 …/lib/lerobot_description/so101_calibration_export_gi_jane.py (see YAML header).
+      Feetech driver reads id, offset, p_cofficient / i_cofficient / d_cofficient (spellings as in driver).
+    -->
     <xacro:property name="use_sim_true" value="${'$(arg use_sim)' in ('true', 'True', '1', 'yes')}"/>
+    <xacro:property name="hw_passive_true" value="${'$(arg hardware_passive)' in ('true', 'True', '1', 'yes')}"/>
+    <xacro:property name="cal" value="${xacro.load_yaml('$(find lerobot_description)/config/so101_follower_calibration.yaml')}"/>
+    <!-- feetech_ros2_driver: joints with no command_interfaces get torque disabled on init. -->
+    <xacro:macro name="feetech_revolute_joint" params="name id offset p:=16 i:=0 d:=32 rd:=0 acc:=254">
+        <joint name="${name}">
+            <param name="id">${id}</param>
+            <param name="offset">${offset}</param>
+            <param name="p_cofficient">${p}</param>
+            <param name="i_cofficient">${i}</param>
+            <param name="d_cofficient">${d}</param>
+            <param name="return_delay_time">${rd}</param>
+            <param name="acceleration">${acc}</param>
+            <xacro:unless value="${hw_passive_true}">
+                <command_interface name="position"/>
+            </xacro:unless>
+            <state_interface name="position"/>
+            <state_interface name="velocity"/>
+        </joint>
+    </xacro:macro>
+    <xacro:macro name="feetech_gripper_joint" params="name id offset p:=16 i:=0 d:=32 rd:=0 acc:=254 mt:=500 pc:=250 ot:=25">
+        <joint name="${name}">
+            <param name="id">${id}</param>
+            <param name="offset">${offset}</param>
+            <param name="p_cofficient">${p}</param>
+            <param name="i_cofficient">${i}</param>
+            <param name="d_cofficient">${d}</param>
+            <param name="return_delay_time">${rd}</param>
+            <param name="acceleration">${acc}</param>
+            <param name="max_torque_limit">${mt}</param>
+            <param name="protection_current">${pc}</param>
+            <param name="overload_torque">${ot}</param>
+            <xacro:unless value="${hw_passive_true}">
+                <command_interface name="position"/>
+            </xacro:unless>
+            <state_interface name="position"/>
+            <state_interface name="velocity"/>
+        </joint>
+    </xacro:macro>
     <xacro:if value="${use_sim_true}">
         <ros2_control name="RobotSystem" type="system">
@@ -61,58 +104,10 @@
                 <param name="usb_port">$(arg usb_port)</param>
             </hardware>
-            <joint name="shoulder_pan">
-                <param name="initial_position">0.0</param>
-                <param name="id">1</param>
-                <param name="p_cofficient">8</param>
-                <param name="offset">-1613</param>
-                <command_interface name="position"/>
-                <state_interface name="position"/>
-                <state_interface name="velocity"/>
-            </joint>
-            <joint name="shoulder_lift">
-                <param name="initial_position">0.0</param>
-                <param name="id">2</param>
-                <param name="p_cofficient">16</param>
-                <param name="offset">-1373</param>
-                <command_interface name="position"/>
-                <state_interface name="position"/>
-                <state_interface name="velocity"/>
-            </joint>
-            <joint name="elbow_flex">
-                <param name="initial_position">0.0</param>
-                <param name="id">3</param>
-                <param name="p_cofficient">16</param>
-                <param name="offset">1681</param>
-                <command_interface name="position"/>
-                <state_interface name="position"/>
-                <state_interface name="velocity"/>
-            </joint>
-            <joint name="wrist_flex">
-                <param name="initial_position">0.0</param>
-                <param name="id">4</param>
-                <param name="p_cofficient">16</param>
-                <param name="offset">-1283</param>
-                <command_interface name="position"/>
-                <state_interface name="position"/>
-                <state_interface name="velocity"/>
-            </joint>
-            <joint name="wrist_roll">
-                <param name="initial_position">0.0</param>
-                <param name="id">5</param>
-                <param name="p_cofficient">16</param>
-                <param name="offset">-471</param>
-                <command_interface name="position"/>
-                <state_interface name="position"/>
-                <state_interface name="velocity"/>
-            </joint>
-            <joint name="gripper_joint">
-                <param name="initial_position">0.0</param>
-                <param name="id">6</param>
-                <param name="p_cofficient">16</param>
-                <param name="offset">-1842</param>
-                <command_interface name="position"/>
-                <state_interface name="position"/>
-                <state_interface name="velocity"/>
-            </joint>
+            <xacro:feetech_revolute_joint name="shoulder_pan" id="${str(cal['joints']['shoulder_pan']['id'])}" offset="${str(cal['joints']['shoulder_pan']['homing_offset'])}" p="${str(cal['joints']['shoulder_pan']['p_coefficient'])}" i="${str(cal['joints']['shoulder_pan']['i_coefficient'])}" d="${str(cal['joints']['shoulder_pan']['d_coefficient'])}" rd="${str(cal['joints']['shoulder_pan']['return_delay_time'])}" acc="${str(cal['joints']['shoulder_pan']['acceleration'])}" />
+            <xacro:feetech_revolute_joint name="shoulder_lift" id="${str(cal['joints']['shoulder_lift']['id'])}" offset="${str(cal['joints']['shoulder_lift']['homing_offset'])}" p="${str(cal['joints']['shoulder_lift']['p_coefficient'])}" i="${str(cal['joints']['shoulder_lift']['i_coefficient'])}" d="${str(cal['joints']['shoulder_lift']['d_coefficient'])}" rd="${str(cal['joints']['shoulder_lift']['return_delay_time'])}" acc="${str(cal['joints']['shoulder_lift']['acceleration'])}" />
+            <xacro:feetech_revolute_joint name="elbow_flex" id="${str(cal['joints']['elbow_flex']['id'])}" offset="${str(cal['joints']['elbow_flex']['homing_offset'])}" p="${str(cal['joints']['elbow_flex']['p_coefficient'])}" i="${str(cal['joints']['elbow_flex']['i_coefficient'])}" d="${str(cal['joints']['elbow_flex']['d_coefficient'])}" rd="${str(cal['joints']['elbow_flex']['return_delay_time'])}" acc="${str(cal['joints']['elbow_flex']['acceleration'])}" />
+            <xacro:feetech_revolute_joint name="wrist_flex" id="${str(cal['joints']['wrist_flex']['id'])}" offset="${str(cal['joints']['wrist_flex']['homing_offset'])}" p="${str(cal['joints']['wrist_flex']['p_coefficient'])}" i="${str(cal['joints']['wrist_flex']['i_coefficient'])}" d="${str(cal['joints']['wrist_flex']['d_coefficient'])}" rd="${str(cal['joints']['wrist_flex']['return_delay_time'])}" acc="${str(cal['joints']['wrist_flex']['acceleration'])}" />
+            <xacro:feetech_revolute_joint name="wrist_roll" id="${str(cal['joints']['wrist_roll']['id'])}" offset="${str(cal['joints']['wrist_roll']['homing_offset'])}" p="${str(cal['joints']['wrist_roll']['p_coefficient'])}" i="${str(cal['joints']['wrist_roll']['i_coefficient'])}" d="${str(cal['joints']['wrist_roll']['d_coefficient'])}" rd="${str(cal['joints']['wrist_roll']['return_delay_time'])}" acc="${str(cal['joints']['wrist_roll']['acceleration'])}" />
+            <xacro:feetech_gripper_joint name="gripper_joint" id="${str(cal['joints']['gripper_joint']['id'])}" offset="${str(cal['joints']['gripper_joint']['homing_offset'])}" p="${str(cal['joints']['gripper_joint']['p_coefficient'])}" i="${str(cal['joints']['gripper_joint']['i_coefficient'])}" d="${str(cal['joints']['gripper_joint']['d_coefficient'])}" rd="${str(cal['joints']['gripper_joint']['return_delay_time'])}" acc="${str(cal['joints']['gripper_joint']['acceleration'])}" mt="${str(cal['joints']['gripper_joint']['max_torque_limit'])}" pc="${str(cal['joints']['gripper_joint']['protection_current'])}" ot="${str(cal['joints']['gripper_joint']['overload_torque'])}" />
         </ros2_control>
     </xacro:unless>
