Commit message: fixng the urdfs and configs to work with the leader arm

File: src/lerobot_description/urdf/so101_base.xacro (robot description, xacro)
@@ -339,15 +339,17 @@
 		</collision>
 	</link>
-	<!-- Joint from gripper to jaw -->
-	<joint name="6" type="revolute">
+	<!-- Joint names align with Hugging Face LeRobot SO-101 (same as servo roles; gripper_joint avoids clashing with link 'gripper'). -->
+	<!-- Joint from gripper link to jaw -->
+	<joint name="gripper_joint" type="revolute">
 		<origin xyz="0.0202 0.0188 -0.0234" rpy="1.5708 -5.14108e-17 -1.38655e-14" />
 		<parent link="gripper" />
 		<child link="jaw" />
 		<axis xyz="0 0 1" />
-		<limit effort="10" velocity="10" lower="-0.174533" upper="1.74533" />
-	</joint>
-	<transmission name="6_trans">
-		<type>transmission_interface/SimpleTransmission</type>
-		<joint name="6">
+		<!-- Commanded full-close ≈ -0.1918 rad; limit slightly beyond for controller margin. -->
+		<limit effort="10" velocity="10" lower="-0.22" upper="1.74533" />
+	</joint>
+	<transmission name="gripper_joint_trans">
+		<type>transmission_interface/SimpleTransmission</type>
+		<joint name="gripper_joint">
 			<hardwareInterface>hardware_interface/PositionJointInterface</hardwareInterface>
 		</joint>
@@ -357,6 +359,6 @@
 		</actuator>
 	</transmission>
-	<!-- Joint from wrist to gripper -->
-	<joint name="5" type="revolute">
+	<!-- Joint from wrist to gripper link -->
+	<joint name="wrist_roll" type="revolute">
 		<origin xyz="0 -0.0611 0.0181" rpy="1.5708 -9.38083e-08 3.14159" />
 		<parent link="wrist" />
@@ -365,7 +367,7 @@
 		<limit effort="10" velocity="10" lower="-2.79253" upper="2.79253" />
 	</joint>
-	<transmission name="5_trans">
-		<type>transmission_interface/SimpleTransmission</type>
-		<joint name="5">
+	<transmission name="wrist_roll_trans">
+		<type>transmission_interface/SimpleTransmission</type>
+		<joint name="wrist_roll">
 			<hardwareInterface>hardware_interface/PositionJointInterface</hardwareInterface>
 		</joint>
@@ -376,5 +378,5 @@
 	</transmission>
 	<!-- Joint from lower_arm to wrist -->
-	<joint name="4" type="revolute">
+	<joint name="wrist_flex" type="revolute">
 		<origin xyz="-0.1349 0.0052 1.65232e-16" rpy="3.2474e-15 2.86219e-15 -1.5708" />
 		<parent link="lower_arm" />
@@ -383,7 +385,7 @@
 		<limit effort="10" velocity="10" lower="-1.65806" upper="1.65806" />
 	</joint>
-	<transmission name="4_trans">
-		<type>transmission_interface/SimpleTransmission</type>
-		<joint name="4">
+	<transmission name="wrist_flex_trans">
+		<type>transmission_interface/SimpleTransmission</type>
+		<joint name="wrist_flex">
 			<hardwareInterface>hardware_interface/PositionJointInterface</hardwareInterface>
 		</joint>
@@ -394,14 +396,15 @@
 	</transmission>
 	<!-- Joint from upper_arm to lower_arm -->
-	<joint name="3" type="revolute">
+	<joint name="elbow_flex" type="revolute">
 		<origin xyz="-0.11257 -0.028 2.46331e-16" rpy="-1.22818e-15 5.75928e-16 1.5708" />
 		<parent link="upper_arm" />
 		<child link="lower_arm" />
 		<axis xyz="0 0 1" />
-		<limit effort="10" velocity="10" lower="-1.74533" upper="1.5708" />
-	</joint>
-	<transmission name="3_trans">
-		<type>transmission_interface/SimpleTransmission</type>
-		<joint name="3">
+		<!-- Limits widened vs stock CAD: leader teleop uses ~−105° / ~+97° body postures after deg→rad -->
+		<limit effort="10" velocity="10" lower="-1.74533" upper="1.85" />
+	</joint>
+	<transmission name="elbow_flex_trans">
+		<type>transmission_interface/SimpleTransmission</type>
+		<joint name="elbow_flex">
 			<hardwareInterface>hardware_interface/PositionJointInterface</hardwareInterface>
 		</joint>
@@ -412,14 +415,14 @@
 	</transmission>
 	<!-- Joint from shoulder to upper_arm -->
-	<joint name="2" type="revolute">
+	<joint name="shoulder_lift" type="revolute">
 		<origin xyz="-0.0303992 -0.0182778 -0.0542" rpy="-1.5708 -1.5708 0" />
 		<parent link="shoulder" />
 		<child link="upper_arm" />
 		<axis xyz="0 0 1" />
-		<limit effort="10" velocity="10" lower="-1.74533" upper="1.74533" />
-	</joint>
-	<transmission name="2_trans">
-		<type>transmission_interface/SimpleTransmission</type>
-		<joint name="2">
+		<limit effort="10" velocity="10" lower="-2.05" upper="1.74533" />
+	</joint>
+	<transmission name="shoulder_lift_trans">
+		<type>transmission_interface/SimpleTransmission</type>
+		<joint name="shoulder_lift">
 			<hardwareInterface>hardware_interface/PositionJointInterface</hardwareInterface>
 		</joint>
@@ -430,5 +433,5 @@
 	</transmission>
 	<!-- Joint from base to shoulder -->
-	<joint name="1" type="revolute">
+	<joint name="shoulder_pan" type="revolute">
 		<origin xyz="0.0207909 -0.0230745 0.0948817" rpy="-3.14159 6.03684e-16 1.5708" />
 		<parent link="base" />
@@ -437,7 +440,7 @@
 		<limit effort="10" velocity="10" lower="-1.91986" upper="1.91986" />
 	</joint>
-	<transmission name="1_trans">
-		<type>transmission_interface/SimpleTransmission</type>
-		<joint name="1">
+	<transmission name="shoulder_pan_trans">
+		<type>transmission_interface/SimpleTransmission</type>
+		<joint name="shoulder_pan">
 			<hardwareInterface>hardware_interface/PositionJointInterface</hardwareInterface>
 		</joint>

File: src/lerobot_description/urdf/so101_ros2_control.xacro (robot description, xacro)
@@ -6,5 +6,5 @@
             <plugin>gz_ros2_control/GazeboSimSystem</plugin>
         </hardware>
-        <joint name="1">
+        <joint name="shoulder_pan">
             <command_interface name="position">
                 <param name="min">-1.91986</param>
@@ -13,19 +13,19 @@
             <state_interface name="position" />
         </joint>
-        <joint name="2">
+        <joint name="shoulder_lift">
             <command_interface name="position">
-                <param name="min">-1.74533</param>
+                <param name="min">-2.05</param>
                 <param name="max">1.74533</param>
             </command_interface>
             <state_interface name="position" />
         </joint>
-        <joint name="3">
+        <joint name="elbow_flex">
             <command_interface name="position">
                 <param name="min">-1.74533</param>
-                <param name="max">1.5708</param>
+                <param name="max">1.85</param>
             </command_interface>
             <state_interface name="position" />
         </joint>
-        <joint name="4">
+        <joint name="wrist_flex">
             <command_interface name="position">
                 <param name="min">-1.65806</param>
@@ -34,5 +34,5 @@
             <state_interface name="position" />
         </joint>
-        <joint name="5">
+        <joint name="wrist_roll">
             <command_interface name="position">
                 <param name="min">-2.79253</param>
@@ -41,7 +41,7 @@
             <state_interface name="position" />
         </joint>
-        <joint name="6">
+        <joint name="gripper_joint">
             <command_interface name="position">
-                <param name="min">-0.174533</param>
+                <param name="min">-0.22</param>
                 <param name="max">1.74533</param>
             </command_interface>

Commit message: Enhance SO101 robot launch and configuration files by adding teleoperation scripts, updating joint limits, and integrating MoveIt Servo for both hardware and simulation environments.

File: src/lerobot_description/urdf/so101_base.xacro (robot description, xacro)
@@ -367,5 +367,6 @@
 		<child link="wrist" />
 		<axis xyz="0 0 1" />
-		<limit effort="10" velocity="10" lower="-1.65806" upper="1.65806" />
+		<!-- Widened from ±1.658 (±95°): leader teleop reaches past stock; avoids Servo limit spam. -->
+		<limit effort="10" velocity="10" lower="-1.74533" upper="1.74533" />
 	</joint>
 	<!-- Joint from upper_arm to lower_arm -->
@@ -384,5 +385,6 @@
 		<child link="upper_arm" />
 		<axis xyz="0 0 1" />
-		<limit effort="10" velocity="10" lower="-2.05" upper="1.74533" />
+		<!-- Lower widened for HW teleop (home ≈ −1.75 rad; stock −2.05 left little “back” travel). -->
+		<limit effort="10" velocity="10" lower="-2.35" upper="1.74533" />
 	</joint>
 	<!-- Joint from base to shoulder -->

File: src/lerobot_description/urdf/so101_ros2_control.xacro (robot description, xacro)
@@ -63,5 +63,5 @@
             <joint name="shoulder_lift">
                 <command_interface name="position">
-                    <param name="min">-2.05</param>
+                    <param name="min">-2.35</param>
                     <param name="max">1.74533</param>
                 </command_interface>
@@ -77,6 +77,6 @@
             <joint name="wrist_flex">
                 <command_interface name="position">
-                    <param name="min">-1.65806</param>
-                    <param name="max">1.65806</param>
+                    <param name="min">-1.74533</param>
+                    <param name="max">1.74533</param>
                 </command_interface>
                 <state_interface name="position"/>

Commit message: Refactor SO101 robot configuration by switching arm and gripper controllers to ForwardCommandController, adding new inertia computation scripts, and integrating Intel RealSense D405 support in URDF. Update simulation settings for MoveIt Servo and enhance launch files for improved teleoperation.

File: src/lerobot_description/urdf/so101_base.xacro (robot description, xacro)
@@ -6,4 +6,9 @@
 -->
 <robot xmlns:xacro="http://www.ros.org/wiki/xacro">
+	<!--
+	  Intel RealSense D405 macro (apt: ros-jazzy-realsense2-description). Defines
+	  the `sensor_d405` xacro macro used below to attach the wrist camera frames.
+	-->
+	<xacro:include filename="$(find realsense2_description)/urdf/_d405.urdf.xacro" />
 	<!-- Links -->
 	<link name="world" />
@@ -281,9 +286,19 @@
 	<!-- Link gripper -->
 	<link name="gripper">
-		<inertial>
-			<origin xyz="0.000213627 0.000245138 -0.025187" rpy="0 0 0" />
-			<mass value="0.087" />
-			<inertia ixx="2.75087e-05" ixy="-3.35241e-07" ixz="-5.7352e-06" iyy="4.33657e-05"
-				iyz="-5.17847e-08" izz="3.45059e-05" />
+		<!--
+		  Inertial composed via scripts/compute_link_inertia.py from:
+		    Wrist_Roll_D405_Holder.stl @ 0.42 g/cm³ (PLA ~20% infill) → 27.31 g holder body,
+		    plus an Intel RealSense D405 modeled as a 60 g uniform 42×42×23 mm box.
+		  TODO(d405-offset): payload xyz is a PLACEHOLDER (0, -0.040, 0.020) m. After
+		  RViz-verifying the holder mesh, measure the D405 body CoM offset on the
+		  holder pocket and re-run compute_link_inertia.py (see its docstring for
+		  the exact command). Wrong payload xyz mostly shows up as wrong off-diagonal
+		  inertia and incorrect CoM along the wrist axis.
+		-->
+		<inertial>
+			<origin xyz="-0.0037735 -0.0295254 0.00594451" rpy="0 0 0" />
+			<mass value="0.087307" />
+			<inertia ixx="9.89785e-05" ixy="9.62938e-06" ixz="-1.42765e-05" iyy="7.30242e-05"
+				iyz="3.28486e-05" izz="6.1257e-05" />
 		</inertial>
 		<!-- Part sts3215_03a_v1_5 -->
@@ -301,5 +316,5 @@
 			</geometry>
 		</collision>
-		<!-- Part wrist_roll_follower_so101_v1 -->
+		<!-- Part Wrist_Roll_D405_Holder (replaces wrist_roll_follower_so101_v1; STL in mm → scale 1e-3). -->
 		<visual>
 			<origin xyz="5.55112e-17 -0.000218214 0.000949706"
@@ -307,5 +322,6 @@
 			<geometry>
 				<mesh
-					filename="package://lerobot_description/meshes/so101/wrist_roll_follower_so101_v1.stl" />
+					filename="package://lerobot_description/meshes/so101/Wrist_Roll_D405_Holder.stl"
+					scale="0.001 0.001 0.001" />
 			</geometry>
 			<material name="3d_printed" />
@@ -316,5 +332,6 @@
 			<geometry>
 				<mesh
-					filename="package://lerobot_description/meshes/so101/wrist_roll_follower_so101_v1.stl" />
+					filename="package://lerobot_description/meshes/so101/Wrist_Roll_D405_Holder.stl"
+					scale="0.001 0.001 0.001" />
 			</geometry>
 		</collision>
@@ -343,4 +360,22 @@
 		</collision>
 	</link>
+	<!--
+	  D405 wrist camera, mounted on the Wrist_Roll_D405_Holder.
+	    parent=gripper          The fixed lower-jaw holder owns the camera.
+	    name=d405_wrist         Frames are d405_wrist_link, d405_wrist_depth_optical_frame, …
+	                            Match this with realsense2_camera's camera_name arg.
+	    use_nominal_extrinsics  Publish nominal datasheet optical extrinsics from the URDF.
+	                            With the live camera, launch realsense2_camera with
+	                            publish_tf:=false so its calibrated frames don't fight.
+	  TODO(d405-mount): replace xyz/rpy below with values measured on the printed
+	  holder. The origin defines gripper → d405_wrist_bottom_screw_frame, where
+	  bottom_screw_frame is the D405's tripod-mount point (bottom centerline of the
+	  camera body) and +X points out the lens. Verify in RViz by toggling the
+	  d405_wrist_link visual: it should sit on the holder's mount pad with the
+	  lens facing the workspace.
+	-->
+	<xacro:sensor_d405 parent="gripper" name="d405_wrist" use_nominal_extrinsics="true">
+		<origin xyz="0.000 -0.096 -0.020" rpy="0.0000 1.0472 1.5708" />
+	</xacro:sensor_d405>
 	<!-- Joint names align with Hugging Face LeRobot SO-101 (same as servo roles; gripper_joint avoids clashing with link 'gripper'). -->
 	<!-- Joint from gripper link to jaw -->

File: src/lerobot_description/urdf/so101_ros2_control.xacro (robot description, xacro)
@@ -50,4 +50,12 @@
     </xacro:macro>
     <xacro:if value="${use_sim_true}">
+        <!--
+          gz_ros2_control reads <param name="initial_value"> on each state_interface
+          to set Gazebo's starting joint pose. Values match initial_positions.yaml
+          (lerobot leader safe-close pose) so the follower in sim starts aligned
+          with the leader at teleop start. Without these, the follower starts at 0
+          while the leader is at ~-100 deg shoulder_lift, which slams MoveIt Servo's
+          AccelerationLimitedPlugin smoother on cycle 1 and produces NaN commands.
+        -->
         <ros2_control name="RobotSystem" type="system">
             <hardware>
@@ -59,5 +67,7 @@
                     <param name="max">1.91986</param>
                 </command_interface>
-                <state_interface name="position"/>
+                <state_interface name="position">
+                    <param name="initial_value">0.090527</param>
+                </state_interface>
             </joint>
             <joint name="shoulder_lift">
@@ -66,5 +76,7 @@
                     <param name="max">1.74533</param>
                 </command_interface>
-                <state_interface name="position"/>
+                <state_interface name="position">
+                    <param name="initial_value">-1.74524</param>
+                </state_interface>
             </joint>
             <joint name="elbow_flex">
@@ -73,5 +85,7 @@
                     <param name="max">1.85</param>
                 </command_interface>
-                <state_interface name="position"/>
+                <state_interface name="position">
+                    <param name="initial_value">1.5708</param>
+                </state_interface>
             </joint>
             <joint name="wrist_flex">
@@ -80,5 +94,7 @@
                     <param name="max">1.74533</param>
                 </command_interface>
-                <state_interface name="position"/>
+                <state_interface name="position">
+                    <param name="initial_value">0.926751</param>
+                </state_interface>
             </joint>
             <joint name="wrist_roll">
@@ -87,5 +103,7 @@
                     <param name="max">2.79253</param>
                 </command_interface>
-                <state_interface name="position"/>
+                <state_interface name="position">
+                    <param name="initial_value">0.278485</param>
+                </state_interface>
             </joint>
             <joint name="gripper_joint">
@@ -94,5 +112,7 @@
                     <param name="max">1.74533</param>
                 </command_interface>
-                <state_interface name="position"/>
+                <state_interface name="position">
+                    <param name="initial_value">-0.191775</param>
+                </state_interface>
             </joint>
         </ros2_control>

Commit message: Add Intel RealSense D405 support by introducing charuco image, updating launch files for staggered hardware bringup, and adding FCC trajectory adapter for MoveIt integration. Enhance configuration files for simulation compatibility and update URDF for D405 wrist camera.

File: src/lerobot_description/urdf/so101_base.xacro (robot description, xacro)
@@ -376,6 +376,7 @@
 	-->
 	<xacro:sensor_d405 parent="gripper" name="d405_wrist" use_nominal_extrinsics="true">
-		<origin xyz="0.000 -0.096 -0.020" rpy="0.0000 1.0472 1.5708" />
+		<origin xyz="0.000 -0.096 -0.020" rpy="0.0000 1.02 1.5708" />
 	</xacro:sensor_d405>
+	<!-- Gazebo rgbd_camera sensor block lives in so101_gazebo.xacro (sim-only file). -->
 	<!-- Joint names align with Hugging Face LeRobot SO-101 (same as servo roles; gripper_joint avoids clashing with link 'gripper'). -->
 	<!-- Joint from gripper link to jaw -->

File: src/lerobot_description/urdf/so101_gazebo.xacro (robot description, xacro)
@@ -7,3 +7,60 @@
         </plugin>
     </gazebo>
+    <!--
+      D405 wrist camera, sim-only sensor block.
+      One rgbd_camera sensor produces four gz topics rooted at /d405_wrist/rgbd:
+        /image           (color, gz.msgs.Image)
+        /depth_image     (float32 depth, gz.msgs.Image)
+        /points          (XYZRGB, gz.msgs.PointCloudPacked)
+        /camera_info     (gz.msgs.CameraInfo)
+      lerobot_description/config/d405_wrist_bridge.yaml remaps these to
+      realsense2_camera-compatible ROS topic names so segmentation / octomap
+      / RViz consumers don't care whether they're talking to sim or hardware.
+      Requires the Sensors system plugin to be loaded by the world SDF —
+      worlds/so101_empty.sdf does that; the stock gz-sim8 empty.sdf does not.
+      optical_frame_id: gz-sim applies the standard ROS optical-frame rotation
+      (image +Z forward, +X right, +Y down) when this is set, so image / depth
+      headers reference d405_wrist_color_optical_frame and downstream nodes
+      don't need an extra static transform.
+    -->
+    <gazebo reference="d405_wrist_link">
+        <sensor name="d405_wrist_rgbd" type="rgbd_camera">
+            <pose>0 0 0 0 0 0</pose>
+            <camera>
+                <!-- D405 datasheet: color ≈ 87° H, depth ≈ 87° H × 58° V; rgbd_camera uses one FOV. -->
+                <horizontal_fov>1.518</horizontal_fov>
+                <!--
+                  Sim resolution intentionally lower than the D405 driver's
+                  default 640x480:
+                    * 320x240 keeps the gz rendering pipeline real-time on the
+                      laptop GPU (640x480 was running ~7 Hz wall-clock).
+                    * Pointcloud becomes ~76k points (~1.2 MB) instead of ~307k
+                      (~5 MB) per frame, so the DDS bridge keeps up at 15 Hz
+                      without dropping packets.
+                  Perception (YOLO-Seg) and octomap care about FOV/intrinsics
+                  more than raw resolution at this stage; we can scale back up
+                  later if needed.
+                -->
+                <image>
+                    <width>320</width>
+                    <height>240</height>
+                </image>
+                <clip>
+                    <!-- D405 sees from ~7 cm; cap depth range at 3 m for sim throughput. -->
+                    <near>0.07</near>
+                    <far>3.0</far>
+                </clip>
+                <optical_frame_id>d405_wrist_color_optical_frame</optical_frame_id>
+            </camera>
+            <always_on>1</always_on>
+            <update_rate>15</update_rate>
+            <topic>d405_wrist/rgbd</topic>
+            <!--
+              Frame ID is set via <optical_frame_id> inside <camera> above.
+              The <gz_frame_id> tag is only valid inside <sensor> for
+              non-camera sensors (IMU, lidar, contact) — gz-sim warns if used
+              for cameras even though it tolerates it. So we omit it here.
+            -->
+        </sensor>
+    </gazebo>
 </robot>
